File: Mini-C3/Mini-C3.kicad_pcb (KiCad board)
At the start: 2 copper layers, 84.1 x 23.3 mm, 30 parts, among them J1 TB_1X2, J10 Sensor1, J11 Sensor1, J12 Sensor1, J2 Sensor1, J3 Sensor1, J4 MotorB, J5 MotorA, J6 Sensor1, J7 Sensor1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

Commit message: panels again
Parts:
- moved G*** 2.55 mm to (156.3, 94.2)
Routing:
- net GND: vias 24 -> 22
Other:
- board text added: "GND"
- board text added: "Vcc"
- board text added: "Vin"
- board text added: "max 4s"
- board text removed: "+"
- board text removed: "Battery"
- board text removed: "Max 4S"

Commit message: silkscreen and gerber files again
Other:
- board text added: "+"
- board text added: "Pinout voltage selector"
- board text removed: "- CAUTION -"
- board text removed: "Select only one (3.3V / 5V) at a time, otherwise, you will fry the board."
- board text removed: "Vcc"
Changed lines of the file:
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@@
 			(outputformat 1)
 			(mirror no)
-			(drillshape 1)
+			(drillshape 0)
 			(scaleselection 1)
-			(outputdirectory "")
+			(outputdirectory "gerber/")
 		)
 	)
@@
 		(tags "switch tactile SPST 1P1T straight NO SMTR C&K")
 		(property "Reference" "SW2"
-			(at 2.2 0.1 -90)
+			(at 0.025 0 0)
 			(unlocked yes)
 			(layer "F.SilkS")
@@
 		(tags "Diode SMA (DO-214AC)")
 		(property "Reference" "D1"
-			(at 0 -2.5 0)
+			(at -3.325 -2.325 180)
 			(layer "F.SilkS")
-			(hide yes)
 			(effects
 				(font
@@
 		(tags "C Disc series Radial pin pitch 5.00mm  diameter 4.3mm width 1.9mm Capacitor")
 		(property "Reference" "C1"
-			(at 2.5 -2.2 0)
+			(at 2.5 0 0)
 			(layer "F.SilkS")
 			(effects
@@
 			(layer "F.Fab")
 		)
-		(fp_text user "${REFERENCE}"
-			(at 2.5 0 0)
-			(layer "F.Fab")
-			(effects
-				(font
-					(size 0.86 0.86)
-					(thickness 0.129)
-				)
-			)
-		)
 		(pad "1" thru_hole circle
 			(at 0 0 180)
@@
 		(at 143.13 94.08 90)
 		(property "Reference" "U3"
-			(at 0 0.5 90)
+			(at 0 0.5 180)
 			(layer "F.SilkS")
-			(hide yes)
 			(effects
 				(font
@@
 		(at 177.85 91.76)
 		(property "Reference" "U1"
-			(at -0.05 12.35 0)
+			(at -0.125 0.24 0)
 			(unlocked yes)
 			(layer "F.SilkS")
-			(hide yes)
 			(effects
 				(font
@@
 		(at 121.23 93.67 90)
 		(property "Reference" "U2"
-			(at -5.715 -13.6525 90)
+			(at 0 0 180)
 			(layer "F.SilkS")
 			(effects
@@
 		(tags "SMD DIP Switch SPST Slide 8.61mm 338mil SMD LowProfile")
 		(property "Reference" "SW3"
-			(at 0 -4.38 90)
+			(at -0.05 -0.075 180)
 			(layer "F.SilkS")
-			(hide yes)
 			(effects
 				(font
@@
 		(tags "solder jumper open")
 		(property "Reference" "JP7"
-			(at 0 1.8 90)
+			(at -0.175 -1.975 90)
 			(layer "B.SilkS")
+			(hide yes)
 			(effects
 				(font
@@
 	(gr_rect
 		(start 166.205 97.7)
-		(end 169.195 100.225)
+		(end 169.42 100.225)
 		(stroke
 			(width 0.1)
 			(type solid)
 		)
-		(fill none)
+		(fill solid)
 		(layer "B.SilkS")
 	)
@@
 		(layer "B.SilkS")
 	)
+	(gr_rect
+		(start 166.21 97.55)
+		(end 169.45 100.225)
+		(stroke
+			(width 0.1)
+			(type solid)
+		)
+		(fill solid)
+		(layer "F.SilkS")
+	)
 	(gr_line
 		(start 192.43 81.82)
@@
 		(layer "Edge.Cuts")
 	)
-	(gr_text "- CAUTION -"
-		(at 141.8 91.4 0)
+	(gr_text "Pinout voltage selector	"
+		(at 141.125 90.8 0)
 		(layer "B.SilkS" knockout)
 		(effects
 			(font
-				(size 1.3 1.3)
-				(thickness 0.2)
+				(size 0.8 0.8)
+				(thickness 0.15)
 				(italic yes)
 			)
@@
 		)
 	)
-	(gr_text "Vcc\n"
-		(at 166.2 102.2 -0)
-		(layer "B.SilkS" knockout)
-		(effects
-			(font
-				(size 1 1)
-				(thickness 0.2)
-				(bold yes)
-			)
-			(justify left bottom mirror)
-		)
-	)
 	(gr_text "JRegi"
 		(at 163.051574 102.525 0)
@@
 	)
 	(gr_text "3.3v"
-		(at 131.5 89.273 -0)
+		(at 131.8 89.7 -0)
 		(layer "B.SilkS" knockout)
 		(effects
@@
 	)
 	(gr_text "5v\n"
-		(at 139.7 89.273 -0)
+		(at 139.35 89.7 -0)
 		(layer "B.SilkS" knockout)
 		(effects
@@
 		)
 	)
-	(gr_text "Select only one (3.3V / 5V) at a time,\notherwise, you will fry the board.\n"
-		(at 149.790478 94.5 0)
-		(layer "B.SilkS" knockout)
-		(effects
-			(font
-				(size 1 1)
-				(thickness 0.15)
-			)
-			(justify left bottom mirror)
-		)
-	)
 	(gr_text "V P6 G"
 		(at 154.4 88.8 0)
@@
 		)
 	)
-	(gr_text "GND"
-		(at 163 99.6 0)
-		(layer "F.SilkS" knockout)
+	(gr_text "-"
+		(at 166.35 98.225 180)
+		(layer "F.SilkS")
 		(effects
 			(font
-				(size 1 1)
-				(thickness 0.2)
+				(size 1.5 1.5)
+				(thickness 0.3)
 				(bold yes)
 			)
@@
 		)
 	)
-	(gr_text "Vin"
-		(at 163.809524 102.2 0)
-		(layer "F.SilkS" knockout)
-		(effects
-			(font
-				(size 1 1)
-				(thickness 0.2)
-				(bold yes)
-			)
-			(justify left bottom)
-		)
-	)
 	(gr_text "V P8 G"
 		(at 162.2 88.9 0)
@@
 		)
 	)
-	(gr_text "-"
-		(at 166.9 97.6 0)
-		(layer "F.SilkS" knockout)
-		(effects
-			(font
-				(size 1 1)
-				(thickness 0.2)
-				(bold yes)
-			)
-			(justify left bottom)
-		)
-	)
 	(gr_text "Vin"
 		(at 157.3 101.5 0)
@@
 				(bold yes)
 			)
+			(justify left bottom)
+		)
+	)
+	(gr_text "+"
+		(at 166.35 100.775 180)
+		(layer "F.SilkS")
+		(effects
+			(font
+				(size 1.5 1.5)
+				(thickness 0.3)
+				(bold yes)
+			)

Commit message: yet another gerber files update
Other:
- board text added: "USB"
Changed lines of the file:
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@@
 		(at 189.35 87.15 -90)
 		(property "Reference" "J5"
-			(at 1.45 5.95 -90)
+			(at 0.25 7.3 -90)
 			(unlocked yes)
 			(layer "F.SilkS")
+			(hide yes)
 			(effects
 				(font
@@
 	)
 	(gr_rect
+		(start 183.4 82.3)
+		(end 185.9 84.6)
+		(stroke
+			(width 0.2)
+			(type solid)
+		)
+		(fill solid)
+		(layer "B.SilkS")
+	)
+	(gr_rect
 		(start 166.205 97.7)
 		(end 169.42 100.225)
@@
 	)
 	(gr_rect
+		(start 170 82.25)
+		(end 172.5 84.55)
+		(stroke
+			(width 0.2)
+			(type solid)
+		)
+		(fill solid)
+		(layer "B.SilkS")
+	)
+	(gr_rect
+		(start 170 82.25)
+		(end 172.5 84.55)
+		(stroke
+			(width 0.2)
+			(type solid)
+		)
+		(fill solid)
+		(layer "F.SilkS")
+	)
+	(gr_rect
+		(start 183.4 82.3)
+		(end 185.9 84.6)
+		(stroke
+			(width 0.2)
+			(type solid)
+		)
+		(fill solid)
+		(layer "F.SilkS")
+	)
+	(gr_rect
 		(start 166.21 97.55)
 		(end 169.45 100.225)
@@
 			)
 			(justify left bottom)
+		)
+	)
+	(gr_text "USB"
+		(at 111.4 95.6 90)
+		(layer "F.SilkS" knockout)
+		(effects
+			(font
+				(size 1.1 1.2)
+				(thickness 0.2)
+				(bold yes)
+			)
+			(justify left bottom)
